File: Pi_HAT/Pi_HAT.kicad_sch (KiCad schematic)
At the start: 17 parts, among them J1 GPIO, J3 AudioJack3, M1 Motor_Servo, U1 TLV2372, U3 ADS1115IDGS

Commit message: sch and pcb done
Parts:
- removed TP1, TP2, TP3: TestPoint, Connector_PinHeader_1.00mm:PinHeader_1x01_P1.00mm_Vertical, symbol Connector:TestPoint
- added JP1: SolderJumper_3_Open, Jumper:SolderJumper-3_P2.0mm_Open_TrianglePad1.0x1.5mm_NumberLabels, symbol Jumper:SolderJumper_3_Open
Connections:
- net SCL1 is gone; now on net GPIO3/SCL1: R6.2, U3.10 (SCL)
- net SDA1 is gone; now on net GPIO2/SDA1: R7.2, U3.9 (SDA)
- new net: JP1.2 (C), U1.3 (+)
- new net: J3.R, JP1.3 (B)
- new net: J3.T, JP1.1 (A)
Changed lines of the file:
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@@
   (junction (at 76.2 43.18) (diameter 1.016) (color 0 0 0 0)
   )
-  (junction (at 91.44 106.68) (diameter 0) (color 0 0 0 0)
-  )
   (junction (at 205.74 90.17) (diameter 0) (color 0 0 0 0)
   )
@@
     (stroke (width 0) (type solid))
   )
-  (wire (pts (xy 91.44 106.68) (xy 91.44 107.95))
-    (stroke (width 0) (type default))
-  )
-  (wire (pts (xy 191.77 116.84) (xy 195.58 116.84))
-    (stroke (width 0) (type default))
-  )
   (wire (pts (xy 218.44 116.84) (xy 218.44 124.46))
     (stroke (width 0) (type default))
@@
     (stroke (width 0) (type solid))
   )
+  (wire (pts (xy 96.52 106.68) (xy 96.52 109.22))
+    (stroke (width 0) (type default))
+  )
   (wire (pts (xy 73.66 76.2) (xy 100.33 76.2))
     (stroke (width 0) (type solid))
@@
     (stroke (width 0) (type solid))
   )
+  (wire (pts (xy 118.11 114.3) (xy 118.11 106.68))
+    (stroke (width 0) (type default))
+  )
+  (wire (pts (xy 91.44 105.41) (xy 93.98 105.41))
+    (stroke (width 0) (type default))
+  )
   (wire (pts (xy 31.75 33.02) (xy 60.96 33.02))
     (stroke (width 0) (type solid))
@@
     (stroke (width 0) (type default))
   )
+  (wire (pts (xy 93.98 105.41) (xy 93.98 106.68))
+    (stroke (width 0) (type default))
+  )
   (wire (pts (xy 31.75 55.88) (xy 60.96 55.88))
     (stroke (width 0) (type solid))
@@
     (stroke (width 0) (type default))
   )
-  (wire (pts (xy 91.44 106.68) (xy 132.08 106.68))
-    (stroke (width 0) (type default))
-  )
   (wire (pts (xy 76.2 24.13) (xy 76.2 27.94))
     (stroke (width 0) (type solid))
@@
     (stroke (width 0) (type default))
   )
+  (wire (pts (xy 100.33 114.3) (xy 118.11 114.3))
+    (stroke (width 0) (type default))
+  )
   (wire (pts (xy 133.35 93.98) (xy 137.16 93.98))
     (stroke (width 0) (type default))
@@
     (stroke (width 0) (type default))
   )
+  (wire (pts (xy 118.11 106.68) (xy 132.08 106.68))
+    (stroke (width 0) (type default))
+  )
   (wire (pts (xy 193.04 90.17) (xy 205.74 90.17))
     (stroke (width 0) (type default))
@@
     (stroke (width 0) (type default))
   )
-  (wire (pts (xy 191.77 114.3) (xy 195.58 114.3))
+  (wire (pts (xy 93.98 106.68) (xy 96.52 106.68))
     (stroke (width 0) (type default))
   )
@@
     (stroke (width 0) (type solid))
   )
+  (wire (pts (xy 91.44 107.95) (xy 91.44 119.38))
+    (stroke (width 0) (type default))
+  )
   (wire (pts (xy 31.75 71.12) (xy 60.96 71.12))
     (stroke (width 0) (type solid))
@@
     (stroke (width 0) (type solid))
   )
-  (wire (pts (xy 91.44 105.41) (xy 91.44 106.68))
-    (stroke (width 0) (type default))
-  )
   (wire (pts (xy 58.42 76.2) (xy 60.96 76.2))
     (stroke (width 0) (type solid))
@@
     (stroke (width 0) (type solid))
   )
+  (wire (pts (xy 91.44 119.38) (xy 96.52 119.38))
+    (stroke (width 0) (type default))
+  )
   (wire (pts (xy 151.13 123.19) (xy 151.13 109.22))
     (stroke (width 0) (type default))
   )
-  (wire (pts (xy 191.77 111.76) (xy 195.58 111.76))
-    (stroke (width 0) (type default))
-  )
   (text "Additional pin functions:\nhttps://pinout.xyz/" (at 179.07 180.34 0)
     (effects (font (size 1.27 1.27)) (justify left bottom))
   )
-  (label "SCL1" (at 231.14 111.76 0) (fields_autoplaced)
-    (effects (font (size 1.27 1.27)) (justify left bottom))
-  )
   (label "ID_SDA" (at 31.75 60.96 0) (fields_autoplaced)
     (effects (font (size 1.27 1.27)) (justify left bottom))
@@
     (effects (font (size 1.27 1.27)) (justify left bottom))
   )
+  (label "GPIO2{slash}SDA1" (at 231.14 114.3 0) (fields_autoplaced)
+    (effects (font (size 1.27 1.27)) (justify left bottom))
+  )
   (label "ID_SCL" (at 100.33 60.96 180) (fields_autoplaced)
     (effects (font (size 1.27 1.27)) (justify right bottom))
@@
     (effects (font (size 1.27 1.27)) (justify left bottom))
   )
+  (label "GPIO3{slash}SCL1" (at 231.14 111.76 0) (fields_autoplaced)
+    (effects (font (size 1.27 1.27)) (justify left bottom))
+  )
   (label "GPIO23" (at 100.33 45.72 180) (fields_autoplaced)
     (effects (font (size 1.27 1.27)) (justify right bottom))
@@
   (label "GPIO7{slash}SPI0.CE1" (at 100.33 58.42 180) (fields_autoplaced)
     (effects (font (size 1.27 1.27)) (justify right bottom))
-  )
-  (label "SDA1" (at 231.14 114.3 0) (fields_autoplaced)
-    (effects (font (size 1.27 1.27)) (justify left bottom))
   )
   (label "GPIO11{slash}SPI0.SCLK" (at 31.75 55.88 0) (fields_autoplaced)
@@
     )
   )
-  (symbol (lib_id "Connector:TestPoint") (at 191.77 116.84 90) (unit 1)
-    (in_bom yes) (on_board yes) (dnp no)
-    (property "Reference" "TP3" (at 185.42 116.84 90)
-      (effects (font (size 1.27 1.27)))
-    )
-    (property "Value" "TestPoint" (at 188.468 114.3 90)
-      (effects (font (size 1.27 1.27)) hide)
-    )
-    (property "Footprint" "Connector_PinHeader_1.00mm:PinHeader_1x01_P1.00mm_Vertical" (at 191.77 111.76 0)
-      (effects (font (size 1.27 1.27)) hide)
-    )
-    (property "Datasheet" "~" (at 191.77 111.76 0)
-      (effects (font (size 1.27 1.27)) hide)
-    )
-    (pin "1")
-    (instances
-      (project "Pi_HAT"
-        (path "/e63e39d7-6ac0-4ffd-8aa3-1841a4541b55"
-          (reference "TP3") (unit 1)
-        )
-      )
-    )
-  )
   (symbol (lib_id "power:GND") (at 205.74 127 0) (unit 1)
     (in_bom yes) (on_board yes) (dnp no)
@@
         (path "/fa2b32db-e4a8-4a65-8bda-51b6f123a044"
           (reference "#PWR0115") (unit 1)
-        )
-      )
-    )
-  )
-  (symbol (lib_id "Connector:TestPoint") (at 191.77 111.76 90) (unit 1)
-    (in_bom yes) (on_board yes) (dnp no)
-    (property "Reference" "TP1" (at 185.42 111.76 90)
-      (effects (font (size 1.27 1.27)))
-    )
-    (property "Value" "TestPoint" (at 188.468 109.22 90)
-      (effects (font (size 1.27 1.27)) hide)
-    )
-    (property "Footprint" "Connector_PinHeader_1.00mm:PinHeader_1x01_P1.00mm_Vertical" (at 191.77 106.68 0)
-      (effects (font (size 1.27 1.27)) hide)
-    )
-    (property "Datasheet" "~" (at 191.77 106.68 0)
-      (effects (font (size 1.27 1.27)) hide)
-    )
-    (pin "1")
-    (instances
-      (project "Pi_HAT"
-        (path "/e63e39d7-6ac0-4ffd-8aa3-1841a4541b55"
-          (reference "TP1") (unit 1)
         )
       )
@@
     )
   )
-  (symbol (lib_id "Connector:TestPoint") (at 191.77 114.3 90) (unit 1)
-    (in_bom yes) (on_board yes) (dnp no)
-    (property "Reference" "TP2" (at 185.42 114.3 90)
-      (effects (font (size 1.27 1.27)))
-    )
-    (property "Value" "TestPoint" (at 188.468 111.76 90)
-      (effects (font (size 1.27 1.27)) hide)
-    )
-    (property "Footprint" "Connector_PinHeader_1.00mm:PinHeader_1x01_P1.00mm_Vertical" (at 191.77 109.22 0)
-      (effects (font (size 1.27 1.27)) hide)
-    )
-    (property "Datasheet" "~" (at 191.77 109.22 0)
-      (effects (font (size 1.27 1.27)) hide)
-    )
-    (pin "1")
-    (instances
-      (project "Pi_HAT"
-        (path "/e63e39d7-6ac0-4ffd-8aa3-1841a4541b55"
-          (reference "TP2") (unit 1)
-        )
-      )
-    )
-  )
   (symbol (lib_id "power:+3.3V") (at 137.16 92.71 0) (unit 1)
     (in_bom yes) (on_board yes) (dnp no)
@@
         )
       )
+    )
+  )
+  (symbol (lib_id "Jumper:SolderJumper_3_Open") (at 96.52 114.3 90) (unit 1)
+    (in_bom yes) (on_board yes) (dnp no)
+    (property "Reference" "JP1" (at 95.25 114.3 90)
+      (effects (font (size 1.27 1.27)) (justify left))
+    )
+    (property "Value" "SolderJumper_3_Open" (at 93.98 120.65 90)
+      (effects (font (size 1.27 1.27)) (justify left))
+    )
+    (property "Footprint" "Jumper:SolderJumper-3_P2.0mm_Open_TrianglePad1.0x1.5mm_NumberLabels" (at 96.52 114.3 0)
+      (effects (font (size 1.27 1.27)) hide)
+    )
+    (property "Datasheet" "~" (at 96.52 114.3 0)
+      (effects (font (size 1.27 1.27)) hide)
+    )
+    (pin "1")
+    (pin "2")
+    (pin "3")
+    (instances
+      (project "Pi_HAT"
+        (path "/e63e39d7-6ac0-4ffd-8aa3-1841a4541b55"
+          (reference "JP1") (unit 1)
+        )
+      )
