File: Pi_HAT/Pi_HAT.kicad_pcb (KiCad board)
At the start: 2 copper layers, 65 x 56 mm, 21 parts, among them J1 GPIO, J3 AudioJack3, M1 Motor_Servo, U1 TLV2372, U3 ADS1115IDGS

Commit message: sch and pcb done
Parts:
- removed TP1, TP2, TP3: TestPoint, Connector_PinHeader_1.00mm:PinHeader_1x01_P1.00mm_Vertical
- added JP1: SolderJumper_3_Open, Jumper:SolderJumper-3_P2.0mm_Open_TrianglePad1.0x1.5mm_NumberLabels, F.Cu at (124.9, 89.6)
- moved R7 34.2 mm to (115.8, 57.0)
- moved R6 31.1 mm to (119.7, 55.8), turned to 180 degrees
- moved C1 28.4 mm to (120.6, 59.7), turned to 90 degrees
- moved U1 28.1 mm to (119.3, 71.3), turned to 90 degrees
- moved U3 27.8 mm to (116.1, 60.1)
- moved R3 27.5 mm to (119.0, 76.7), turned to 90 degrees
- moved C3 27.4 mm to (118.2, 66.1)
- moved D1 27.3 mm to (113.9, 72.7), turned to -90 degrees
- moved R5 27.3 mm to (111.5, 76.7), turned to 90 degrees
- moved R4 26.9 mm to (116.5, 75.9)
- moved C2 20.4 mm to (113.7, 77.5), turned to -90 degrees
- moved J3 4.46 mm to (116.0, 90.9), turned to 180 degrees
Connections:
- J3 pad R: Net-(U1A-+) -> Net-(JP1-B)
- J3 pad T: Net-(U1A-+) -> Net-(JP1-A)
- R6 pad 2: /SCL1 -> /GPIO3/SCL1
- R7 pad 2: /SDA1 -> /GPIO2/SDA1
- U1 pad 3: Net-(U1A-+) -> Net-(JP1-C)
- U3 pad 10: /SCL1 -> /GPIO3/SCL1
- U3 pad 5: Net-(U3-AIN1) -> unconnected-(U3-AIN1-Pad5)
- U3 pad 6: Net-(U3-AIN2) -> unconnected-(U3-AIN2-Pad6)
- U3 pad 7: Net-(U3-AIN3) -> unconnected-(U3-AIN3-Pad7)
- U3 pad 9: /SDA1 -> /GPIO2/SDA1
Routing:
- net +5V: track 0.00 -> 71.4 mm
- net /GPIO12/PWM0: track 0.00 -> 59.9 mm
- net +3V3: track 0.00 -> 36.1 mm
- net Net-(JP1-C): track 0.00 -> 21.4 mm
- net /ENVELOPE_OUT: track 0.00 -> 19.5 mm
- net /GPIO2/SDA1: track 0.00 -> 15.1 mm
- net /GPIO3/SCL1: track 0.00 -> 13.3 mm
- net Net-(JP1-B): track 0.00 -> 12.9 mm
- net Net-(D1-A): track 0.00 -> 6.18 mm
- net Net-(JP1-A): track 0.00 -> 6.10 mm
- net Net-(U1A--): track 0.00 -> 4.08 mm
- net GND: track 0.00 -> 1.82 mm
- added copper zone on F.Cu, net GND
Other:
- board text added: "To OpAmp"

Commit message: added some final bits - silk etc
Other:
- board text added: "e-NT"
